Commit message: Invert the right legs and the left legs

File: urdf/phantomx.urdf (robot description, URDF)
Before this commit: robot PhantomX, 26 links, 25 joints
Joints:
- joint j_c1_lf: origin xyz=0.1248 -0.06164  0.001116 rpy=0 4.7123 0.7853981633974483 -> xyz=0.1248 0.06164  0.001116 rpy=0 4.7123 2.356194490192345
- joint j_c1_lm: origin xyz=0 -0.1034  0.001116 rpy=0 4.7123 0 -> xyz=0 0.1034  0.001116 rpy=0 4.7123 3.14159
- joint j_c1_lr: origin xyz=-0.1248 -0.06164  0.001116 rpy=0 4.7123 -0.7853981633974483 -> xyz=-0.1248 0.06164  0.001116 rpy=0 4.7123 3.9269908169872414
- joint j_c1_rf: origin xyz=0.1248 0.06164  0.001116 rpy=0 4.7123 2.356194490192345 -> xyz=0.1248 -0.06164  0.001116 rpy=0 4.7123 0.7853981633974483
- joint j_c1_rm: origin xyz=0 0.1034  0.001116 rpy=0 4.7123 3.14159 -> xyz=0 -0.1034  0.001116 rpy=0 4.7123 0
- joint j_c1_rr: origin xyz=-0.1248 0.06164  0.001116 rpy=0 4.7123 3.9269908169872414 -> xyz=-0.1248 -0.06164  0.001116 rpy=0 4.7123 -0.7853981633974483
- joint j_thigh_lf: origin xyz=0 0 0 rpy= 0 3.14159 3.14159 -> xyz=0 0 0 rpy=3.14159 0  0
- joint j_thigh_lm: origin xyz=0 0 0 rpy= 0 3.14159 3.14159 -> xyz=0 0 0 rpy=3.14159 0  0
- joint j_thigh_lr: origin xyz=0 0 0 rpy= 0 3.14159 3.14159 -> xyz=0 0 0 rpy=3.14159 0  0
- joint j_thigh_rf: origin xyz=0 0 0 rpy= 0 3.14159 3.14159 -> xyz=0 0 0 rpy=3.14159 0  0
- joint j_thigh_rm: origin xyz=0 0 0 rpy= 0 3.14159 3.14159 -> xyz=0 0 0 rpy=3.14159 0  0
- joint j_thigh_rr: origin xyz=0 0 0 rpy= 0 3.14159 3.14159 -> xyz=0 0 0 rpy=3.14159 0  0

File: urdf/phantomx_urdf.xacro (robot description, xacro)
@@ -37,10 +37,10 @@
         <material>Gazebo/Grey</material>
       </gazebo>
-    <xacro:leg_l xyz="0.1248 -0.06164  0.001116"  rpy="0 4.7123 0.7853981633974483" suffix="lf"/>
-    <xacro:leg_l xyz="0 -0.1034  0.001116"  rpy="0 4.7123 0" suffix="lm"/>
-    <xacro:leg_l xyz="-0.1248 -0.06164  0.001116"  rpy="0 4.7123 -0.7853981633974483" suffix="lr"/>
-    <xacro:leg_l xyz="0.1248 0.06164  0.001116"  rpy="0 4.7123 2.356194490192345" suffix="rf"/>
-    <xacro:leg_l xyz="0 0.1034  0.001116"  rpy="0 4.7123 3.14159" suffix="rm"/>
-    <xacro:leg_l xyz="-0.1248 0.06164  0.001116"  rpy="0 4.7123 3.9269908169872414" suffix="rr"/>
+    <xacro:leg_l xyz="0.1248 -0.06164  0.001116"  rpy="0 4.7123 0.7853981633974483" suffix="rf"/>
+    <xacro:leg_l xyz="0 -0.1034  0.001116"  rpy="0 4.7123 0" suffix="rm"/>
+    <xacro:leg_l xyz="-0.1248 -0.06164  0.001116"  rpy="0 4.7123 -0.7853981633974483" suffix="rr"/>
+    <xacro:leg_l xyz="0.1248 0.06164  0.001116"  rpy="0 4.7123 2.356194490192345" suffix="lf"/>
+    <xacro:leg_l xyz="0 0.1034  0.001116"  rpy="0 4.7123 3.14159" suffix="lm"/>
+    <xacro:leg_l xyz="-0.1248 0.06164  0.001116"  rpy="0 4.7123 3.9269908169872414" suffix="lr"/>
 </xacro:macro>
  <xacro:macro name="leg_l" params="xyz rpy suffix">
