Commit message: Work Complete. Closed.

File: urdf/autogen_phantomx.urdf (robot description, URDF)
Before this commit: robot PhantomX, 26 links, 25 joints
Joints:
- joint j_thigh_lf: origin xyz=0 0 0 rpy=3.14159 0  0 -> xyz=0 0 0 rpy= 0 3.14159 3.14159
- joint j_thigh_lm: origin xyz=0 0 0 rpy=3.14159 0  0 -> xyz=0 0 0 rpy= 0 3.14159 3.14159
- joint j_thigh_lr: origin xyz=0 0 0 rpy=3.14159 0  0 -> xyz=0 0 0 rpy= 0 3.14159 3.14159
- joint j_thigh_rf: origin xyz=0 0 0 rpy=3.14159 0  0 -> xyz=0 0 0 rpy= 0 3.14159 3.14159
- joint j_thigh_rm: origin xyz=0 0 0 rpy=3.14159 0  0 -> xyz=0 0 0 rpy= 0 3.14159 3.14159
- joint j_thigh_rr: origin xyz=0 0 0 rpy=3.14159 0  0 -> xyz=0 0 0 rpy= 0 3.14159 3.14159

File: urdf/phantomx_urdf.xacro (robot description, xacro)
@@ -4,4 +4,7 @@
 <xacro:property name="thigh_offset_y" value="-0.0645" />
 <xacro:property name="thigh_offset_z" value="-0.0145" />
+<xacro:property name="body_color" value="Gazebo/Red" />
+<xacro:property name="tibia_color" value="Gazebo/Green" />
+<xacro:property name="thigh_color" value="Gazebo/Blue" />
 <xacro:macro name="phantomx" params="parent *origin">
       <joint name="j_phantomx_attachment" type="fixed">
@@ -23,7 +26,4 @@
             <mesh filename="package://phantomx_description/meshes/body.STL"  scale="1 1 1"/>
           </geometry>
-          <material name="Grey">
-            <color rgba="0.20 0.20 0.20 1.0"/>
-          </material>
         </visual>
         <collision>
@@ -35,5 +35,5 @@
       </link>
       <gazebo reference="MP_BODY">
-        <material>Gazebo/Grey</material>
+        <material>${body_color}</material>
       </gazebo>
     <xacro:leg_l xyz="0.1248 -0.06164  0.001116"  rpy="0 4.7123 0.7853981633974483" suffix="rf"/>
@@ -57,7 +57,4 @@
         <mesh filename="package://phantomx_description/meshes/connect.STL"  scale="1 1 1"/>
       </geometry>
-      <material name="Grey">
-        <color rgba="0.20 0.20 0.20 1.0"/>
-      </material>
     </visual>
     <collision>
@@ -80,7 +77,4 @@
         <mesh filename="package://phantomx_description/meshes/connect.STL"  scale="1 1 1"/>
       </geometry>
-      <material name="Grey">
-        <color rgba="0.20 0.20 0.20 1.0"/>
-      </material>
     </visual>
     <collision>
@@ -103,7 +97,4 @@
         <mesh filename="package://phantomx_description/meshes/thigh_l.STL"  scale="1 1 1"/>
       </geometry>
-      <material name="Grey">
-        <color rgba="0.20 0.20 0.20 1.0"/>
-      </material>
     </visual>
     <collision>
@@ -126,7 +117,4 @@
         <mesh filename="package://phantomx_description/meshes/tibia_l.STL"  scale="1 1 1"/>
       </geometry>
-      <material name="Grey">
-        <color rgba="0.20 0.20 0.20 1.0"/>
-      </material>
     </visual>
     <collision>
@@ -194,14 +182,14 @@
   </transmission>
   <gazebo reference="c1_${suffix}">
-    <material>Gazebo/Grey</material>
+    <material>${body_color}</material>
   </gazebo>
   <gazebo reference="c2_${suffix}">
-    <material>Gazebo/Grey</material>
+    <material>${thigh_color}</material>
   </gazebo>
   <gazebo reference="thigh_${suffix}">
-    <material>Gazebo/Grey</material>
+    <material>${thigh_color}</material>
   </gazebo>
   <gazebo reference="tibia_${suffix}">
-    <material>Gazebo/Grey</material>
+    <material>${tibia_color}</material>
   </gazebo>
 </xacro:macro>

Commit message: Work Complete. Closed.

File: urdf/autogen_phantomx.urdf (robot description, URDF)
Before this commit: robot PhantomX, 26 links, 25 joints
Links:
- link MP_BODY: mass 0.97559947 -> 5

File: urdf/phantomx_urdf.xacro (robot description, xacro)
@@ -16,5 +16,5 @@
         <inertial>
           <origin xyz="0 0 0" />
-          <mass value="0.97559947"/>
+          <mass value="5"/>
           <inertia ixx="3.1081800"  ixy="-0.25460189"  ixz="2.0318174" iyy="6.3787776" iyz="0.16417863" izz="5.3316425" />
         </inertial>
